File: BatteryManagment/BatteryManagment.kicad_sch (KiCad schematic)
At the start: 0 parts

Commit message: fixed temperature sensor, BMS schematic done
Parts:
- added C1, C2: 1uF, Capacitor_SMD:C_0603_1608Metric_Pad1.08x0.95mm_HandSolder, symbol Device:C
- added J1, J2: Conn_01x02_Pin, Connector_JST:JST_EH_S2B-EH_1x02_P2.50mm_Horizontal, symbol Connector:Conn_01x02_Pin
- added J3: PT1000, Connector_JST:JST_EH_S2B-EH_1x02_P2.50mm_Horizontal, symbol Connector:Conn_01x02_Pin
- added R1, R2, R3, R4, R5, R6, R7: R, Resistor_SMD:R_0603_1608Metric_Pad0.98x0.95mm_HandSolder, symbol Device:R
- added U1: BQ25176MDSGR, footprints:WSON_MDSGR_TEX, symbol SensorNode:BQ25176MDSGR
- added U2: Opamp_Dual, symbol Device:Opamp_Dual
Connections:
- new net: J3.1 (Pin_1), R4.2, U2.2 (-), U2.3 (+), U2.5 (+), U2.6 (-)
- new net: R5.2, U2.1, U2.7
- new net: R1.2, R2.1
- new net: R2.2, R3.1
- new net: C1.1, J1.1 (Pin_1), R1.1, R4.1, R5.1, U1.1 (IN), U2.8 (V+)
- new net: C1.2, C2.2, J1.2 (Pin_2), J2.2 (Pin_2), J3.2 (Pin_2), R3.2, R6.2, R7.2, U1.4 (GND), U1.9 (GND), U2.4 (V-)
- new net: R7.1, U1.7 (VSET)
- new net: R6.1, U1.2 (ISET)
- new net: C2.1, J2.1 (Pin_1), U1.8 (OUT)
- no-connect marks 0 -> 3
